File: ps2-tatacon-rp2040.kicad_pcb (KiCad board)
At the start: 2 copper layers, 50 x 35 mm, 4 parts

Commit message: Board layout finished, need to fix footprint
Parts:
- removed REF**: BUTTONS, Connector_PinSocket_2.54mm:PinSocket_1x03_P2.54mm_Vertical
- removed REF**: RIGHT, tatacon_connectors:PinSocket_1x02_Spaced_P2.00mm
- removed REF**: LEFT, tatacon_connectors:PinSocket_1x02_Spaced_P2.00mm
- removed REF**: CENTER, tatacon_connectors:PinSocket_1x04_P2.5mm_Vertical
- added C1: 100nF, Capacitor_SMD:C_0603_1608Metric_Pad1.08x0.95mm_HandSolder, F.Cu at (57.7, 26.4)
- added C2: 100nF, Capacitor_SMD:C_0603_1608Metric_Pad1.08x0.95mm_HandSolder, F.Cu at (33.4, 39.2)
- added C3: 100nF, Capacitor_SMD:C_0603_1608Metric_Pad1.08x0.95mm_HandSolder, F.Cu at (35.9, 48.6)
- added C4: 100nF, Capacitor_SMD:C_0603_1608Metric_Pad1.08x0.95mm_HandSolder, F.Cu at (47.0, 53.1)
- added J1: Buttons, Connector_PinSocket_2.54mm:PinSocket_1x03_P2.54mm_Vertical, F.Cu at (40.2, 27.9)
- added J2: Right, tatacon_connectors:PinSocket_1x02_Spaced_P2.00mm, F.Cu at (63.0, 26.4)
- added J3: Left, tatacon_connectors:PinSocket_1x02_Spaced_P2.00mm, F.Cu at (38.7, 39.2)
- added J4: Center, tatacon_connectors:PinSocket_1x04_P2.5mm_Vertical, F.Cu at (41.1, 48.6)
- added R1: 50K, Resistor_SMD:R_0603_1608Metric_Pad0.98x0.95mm_HandSolder, F.Cu at (42.0, 32.4)
- added R2: 50K, Resistor_SMD:R_0603_1608Metric_Pad0.98x0.95mm_HandSolder, F.Cu at (46.1, 32.4)
- added R3: 50K, Resistor_SMD:R_0603_1608Metric_Pad0.98x0.95mm_HandSolder, F.Cu at (57.7, 29.3)
- added R4: 50K, Resistor_SMD:R_0603_1608Metric_Pad0.98x0.95mm_HandSolder, F.Cu at (33.4, 42.2)
- added R5: 50K, Resistor_SMD:R_0603_1608Metric_Pad0.98x0.95mm_HandSolder, F.Cu at (35.9, 51.1)
- added R6: 50K, Resistor_SMD:R_0603_1608Metric_Pad0.98x0.95mm_HandSolder, F.Cu at (47.0, 55.6)
- added U1: RP2040-Zero, RP2040-Zero-Kicad:RP2040-Zero, F.Cu at (53.4, 31.5)
Routing:
- net L_KA: track 0.00 -> 7.46 mm
- net R_KA: track 0.00 -> 7.41 mm
- net R_DON: track 0.00 -> 6.97 mm
- net L_DON: track 0.00 -> 6.96 mm
- net SELECT: track 0.00 -> 4.57 mm
- net START: track 0.00 -> 4.57 mm
- added copper zone on F.Cu, net GND

Commit message: First revision finished
Parts:
- added REF**: blob, exentio_art:exentio_blob, F.Cu at (33.0, 34.0)
- moved C4 1.77 mm to (45.2, 53.1), turned to 180 degrees
- moved R6 1.77 mm to (45.2, 55.6), turned to 0 degrees
Connections:
- U1 pad 14: unconnected-(U1-GP13-Pad14) -> START
- U1 pad 15: START -> SELECT
- U1 pad 7: unconnected-(U1-GP6-Pad7) -> R_DON
- U1 pad 8: unconnected-(U1-GP7-Pad8) -> L_DON
Routing:
- net +3.3V: track 0.00 -> 88.9 mm, vias 0 -> 4
- net L_KA: track 7.46 -> 44.0 mm, vias 0 -> 1
- net L_DON: track 6.96 -> 26.9 mm, vias 0 -> 1
- net SELECT: track 4.57 -> 21.9 mm
- net R_DON: track 6.97 -> 23.8 mm
- net START: track 4.57 -> 19.9 mm
- net R_KA: track 7.41 -> 16.9 mm
- added copper zone on B.Cu, net GND
Other:
- board text added: "DO NOT PLACE HERE"
- board text added: "PS2 Tatacon (NPC-107) RP2040 Adapter v1 by Exentio Kawasaki"
